File: NightLight.kicad_pcb (KiCad board)
At the start: 2 copper layers, 99.4 x 86.1 mm, 29 parts, among them J1 Conn_01x02, J2 Micro_SD_Card, J3 TTL, J5 Touch1, J6 Touch2, SW1 POWER-ON, SW2 SW_Push, U1 magnetic-charger, U2 rdm-6300, U3 TP4056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

Commit message: Minor changes
Parts:
- moved J2 0.70 mm to (100.7, 139.7)
Routing:
- net GND: track 55.2 -> 57.1 mm
- net RFID_TX: track 35.9 -> 36.6 mm
- net MOSI: track 52.8 -> 52.1 mm
- net MISO: track 75.6 -> 74.9 mm
Changed lines of the file:
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@@
     (property "Sheetname" "")
     (attr exclude_from_pos_files)
-    (fp_text reference "H2" (at 0 -6.3) (layer "F.SilkS")
-      (effects (font (size 1 1) (thickness 0.15)))
-    )
-    (fp_text value "MountingHole" (at 0 6.3) (layer "F.Fab")
-      (effects (font (size 1 1) (thickness 0.15)))
-    )
-    (fp_text user "${REFERENCE}" (at 0 0) (layer "F.Fab")
+    (fp_text reference "H2" (at 4 -34.3) (layer "F.SilkS")
+      (effects (font (size 1 1) (thickness 0.15)))
+    )
+    (fp_text value "MountingHole" (at 4.5 -30.3) (layer "F.Fab")
+      (effects (font (size 1 1) (thickness 0.15)))
+    )
+    (fp_text user "${REFERENCE}" (at 2.7 -37.2) (layer "F.Fab")
       (effects (font (size 1 1) (thickness 0.15)))
     )
@@
   )
   (footprint "sd-card:sd-card" (layer "F.Cu")
-    (at 100.7 140.4 90)
+    (at 100.7 139.7 90)
     (property "Sheetfile" "NightLight.kicad_sch")
     (property "Sheetname" "")
@@
     (pad "25" smd rect (at 8.5 -8.255 240) (size 2 0.9) (layers "B.Cu" "B.Paste" "B.Mask")
       (net 20 "BOOT") (pinfunction "IO0") (pintype "bidirectional"))
-    (pad "26" smd rect (at 8.5 -6.985 240) (size 3 0.9) (layers "B.Cu" "B.Paste" "B.Mask")
+    (pad "26" smd rect (at 8.5 -6.985 240) (size 2.5 0.9) (layers "B.Cu" "B.Paste" "B.Mask")
       (net 31 "unconnected-(U4-Pad26)") (pinfunction "IO4") (pintype "bidirectional"))
     (pad "27" smd rect (at 8.5 -5.715 240) (size 3 0.9) (layers "B.Cu" "B.Paste" "B.Mask")
@@
     (pad "31" smd rect (at 8.5 -0.635 240) (size 3 0.9) (layers "B.Cu" "B.Paste" "B.Mask")
       (net 8 "RFID_LED") (pinfunction "IO19") (pintype "bidirectional"))
-    (pad "32" smd rect (at 8.5 0.635 240) (size 3 0.9) (layers "B.Cu" "B.Paste" "B.Mask")
+    (pad "32" smd rect (at 8.5 0.635 240) (size 2 0.9) (layers "B.Cu" "B.Paste" "B.Mask")
       (net 36 "unconnected-(U4-Pad32)") (pinfunction "NC") (pintype "no_connect"))
     (pad "33" smd rect (at 8.5 1.905 240) (size 2 0.9) (layers "B.Cu" "B.Paste" "B.Mask")
@@
     (pad "35" smd rect (at 8.5 4.445 240) (size 2 0.9) (layers "B.Cu" "B.Paste" "B.Mask")
       (net 33 "TX") (pinfunction "TXD0/IO1") (pintype "bidirectional"))
-    (pad "36" smd rect (at 8.5 5.715 240) (size 3 0.9) (layers "B.Cu" "B.Paste" "B.Mask")
+    (pad "36" smd rect (at 8.5 5.715 240) (size 3.5 0.9) (layers "B.Cu" "B.Paste" "B.Mask")
       (net 39 "unconnected-(U4-Pad36)") (pinfunction "IO22") (pintype "bidirectional"))
-    (pad "37" smd rect (at 8.5 6.985 240) (size 3 0.9) (layers "B.Cu" "B.Paste" "B.Mask")
+    (pad "37" smd rect (at 8.5 6.985 240) (size 3.5 0.9) (layers "B.Cu" "B.Paste" "B.Mask")
       (net 35 "unconnected-(U4-Pad37)") (pinfunction "IO23") (pintype "bidirectional"))
     (pad "38" smd rect (at 8.5 8.255 240) (size 3 0.9) (layers "B.Cu" "B.Paste" "B.Mask")
@@
   (segment (start 82.51 67.71) (end 84 69.2) (width 1) (layer "B.Cu") (net 6))
   (segment (start 87.5 101) (end 86.7 100.2) (width 1) (layer "B.Cu") (net 6))
+  (segment (start 70.4 68.6) (end 70.4 69.9) (width 1) (layer "B.Cu") (net 6))
   (segment (start 101.5 63.1) (end 102.47 63.1) (width 1) (layer "B.Cu") (net 6))
+  (segment (start 70.4 69.9) (end 70.8 70.3) (width 1) (layer "B.Cu") (net 6))
   (segment (start 82.51 66.04) (end 82.51 67.71) (width 1) (layer "B.Cu") (net 6))
   (segment (start 80.449501 124.994127) (end 82.903037 122.540591) (width 0.1) (layer "F.Cu") (net 7))
@@
   (segment (start 86.878679 110) (end 88.294971 110) (width 0.6) (layer "B.Cu") (net 19))
   (segment (start 85.3 105.1) (end 86 105.8) (width 0.6) (layer "B.Cu") (net 19))
-  (segment (start 96.7 140.4) (end 96.7 136.75) (width 0.6) (layer "B.Cu") (net 19))
+  (segment (start 90.8 129.138667) (end 89.600499 127.939166) (width 0.6) (layer "B.Cu") (net 19))
+  (segment (start 96.7 136.75) (end 90.8 130.85) (width 0.6) (layer "B.Cu") (net 19))
+  (segment (start 96.7 139.7) (end 96.7 136.75) (width 0.6) (layer "B.Cu") (net 19))
+  (segment (start 89.600499 120.599501) (end 90.685747 119.514253) (width 0.6) (layer "B.Cu") (net 19))
   (segment (start 90.8 130.85) (end 90.8 129.138667) (width 0.6) (layer "B.Cu") (net 19))
-  (segment (start 89.600499 120.599501) (end 90.685747 119.514253) (width 0.6) (layer "B.Cu") (net 19))
-  (segment (start 90.8 129.138667) (end 89.600499 127.939166) (width 0.6) (layer "B.Cu") (net 19))
   (segment (start 86 105.8) (end 86 109.121321) (width 0.6) (layer "B.Cu") (net 19))
-  (segment (start 96.7 136.75) (end 90.8 130.85) (width 0.6) (layer "B.Cu") (net 19))
   (segment (start 88.294971 110) (end 90.170526 111.875555) (width 0.6) (layer "B.Cu") (net 19))
   (segment (start 83 102) (end 83 108.5) (width 0.6) (layer "F.Cu") (net 20))
@@
   (via (at 86.6 113.1) (size 2.5) (drill 0.8) (layers "F.Cu" "B.Cu") (net 21))
   (via (at 87.1 119.1) (size 2.5) (drill 0.8) (layers "F.Cu" "B.Cu") (net 21))
-  (segment (start 71.861134 105.853183) (end 71.861134 105.544291) (width 0.6) (layer "B.Cu") (net 21))
-  (segment (start 84.4505 110.5505) (end 76.558451 110.5505) (width 0.6) (layer "B.Cu") (net 21))
+  (segment (start 71.861134 107.161134) (end 71.861134 105.544291) (width 0.6) (layer "B.Cu") (net 21))
+  (segment (start 90.000499 131.771164) (end 90.000499 129.469832) (width 0.6) (layer "B.Cu") (net 21))
+  (segment (start 90.000499 129.469832) (end 88.8 128.269333) (width 0.6) (layer "B.Cu") (net 21))
   (segment (start 94.7 136.470665) (end 90.000499 131.771164) (width 0.6) (layer "B.Cu") (net 21))
   (segment (start 71.861134 105.544291) (end 72.593184 104.812241) (width 0.6) (layer "B.Cu") (net 21))
+  (segment (start 84.4505 110.5505) (end 75.2505 110.5505) (width 0.6) (layer "B.Cu") (net 21))
+  (segment (start 94.7 139.7) (end 94.7 136.470665) (width 0.6) (layer "B.Cu") (net 21))
+  (segment (start 88.8 128.269333) (end 88.8 120.303112) (width 0.6) (layer "B.Cu") (net 21))
+  (segment (start 87.232786 112.463452) (end 87.232786 112.7495) (width 0.6) (layer "B.Cu") (net 21))
   (segment (start 88.8 120.303112) (end 87.9 119.403112) (width 0.6) (layer "B.Cu") (net 21))
-  (segment (start 90.000499 129.469832) (end 88.8 128.269333) (width 0.6) (layer "B.Cu") (net 21))
-  (segment (start 94.7 140.4) (end 94.7 136.470665) (width 0.6) (layer "B.Cu") (net 21))
-  (segment (start 90.000499 131.771164) (end 90.000499 129.469832) (width 0.6) (layer "B.Cu") (net 21))
-  (segment (start 88.8 128.269333) (end 88.8 120.303112) (width 0.6) (layer "B.Cu") (net 21))
+  (segment (start 75.2505 110.5505) (end 71.861134 107.161134) (width 0.6) (layer "B.Cu") (net 21))
   (segment (start 86.6 112.7) (end 84.4505 110.5505) (width 0.6) (layer "B.Cu") (net 21))
-  (segment (start 87.232786 112.463452) (end 87.232786 112.7495) (width 0.6) (layer "B.Cu") (net 21))
-  (segment (start 76.558451 110.5505) (end 71.861134 105.853183) (width 0.6) (layer "B.Cu") (net 21))
   (segment (start 111.76 123.19) (end 111.76 136.1495) (width 0.6) (layer "F.Cu") (net 30))
   (via (at 111.76 123.19) (size 2.5) (drill 0.8) (layers "F.Cu" "B.Cu") (net 30))
   (via (at 111.76 136.1495) (size 2.5) (drill 0.8) (layers "F.Cu" "B.Cu") (net 30))
   (segment (start 92.744173 115) (end 77.395168 115) (width 0.6) (layer "B.Cu") (net 30))
-  (segment (start 104.7 140.4) (end 104.7 138.5) (width 0.6) (layer "B.Cu") (net 30))
   (segment (start 77.395168 115) (end 69.66143 107.266262) (width 0.6) (layer "B.Cu") (net 30))
   (segment (start 69.66143 104.274291) (end 70.39348 103.542241) (width 0.6) (layer "B.Cu") (net 30))
   (segment (start 69.66143 107.266262) (end 69.66143 104.274291) (width 0.6) (layer "B.Cu") (net 30))
+  (segment (start 104.7 138.5) (end 107.0505 136.1495) (width 0.6) (layer "B.Cu") (net 30))
   (segment (start 107.0505 136.1495) (end 111.76 136.1495) (width 0.6) (layer "B.Cu") (net 30))
-  (segment (start 104.7 138.5) (end 107.0505 136.1495) (width 0.6) (layer "B.Cu") (net 30))
   (segment (start 100.934173 123.19) (end 92.744173 115) (width 0.6) (layer "B.Cu") (net 30))
   (segment (start 111.76 123.19) (end 100.934173 123.19) (width 0.6) (layer "B.Cu") (net 30))
+  (segment (start 104.7 139.7) (end 104.7 138.5) (width 0.6) (layer "B.Cu") (net 30))
   (segment (start 64.60436 101.850374) (end 64.894218 102.140232) (width 0.6) (layer "B.Cu") (net 32))
   (segment (start 62.55 106.15) (end 58.75 106.15) (width 0.6) (layer "B.Cu") (net 32))
@@
   (via (at 78.698843 122.988686) (size 2.5) (drill 0.8) (layers "F.Cu" "B.Cu") (net 52))
   (via (at 78.7 112.7) (size 2.5) (drill 0.8) (layers "F.Cu" "B.Cu") (net 52))
+  (segment (start 76.269335 112.7) (end 78.7 112.7) (width 0.6) (layer "B.Cu") (net 52))
   (segment (start 71.493332 104.177241) (end 70.761282 104.909291) (width 0.6) (layer "B.Cu") (net 52))
   (segment (start 86.686316 130.976159) (end 78.698843 122.988686) (width 0.6) (layer "B.Cu") (net 52))
-  (segment (start 70.761282 104.909291) (end 70.761282 105.883996) (width 0.6) (layer "B.Cu") (net 52))
-  (segment (start 70.761282 105.883996) (end 77.577286 112.7) (width 0.6) (layer "B.Cu") (net 52))
+  (segment (start 70.761282 107.191947) (end 76.269335 112.7) (width 0.6) (layer "B.Cu") (net 52))
   (segment (start 88.208228 130.976159) (end 86.686316 130.976159) (width 0.6) (layer "B.Cu") (net 52))
-  (segment (start 77.577286 112.7) (end 78.7 112.7) (width 0.6) (layer "B.Cu") (net 52))
+  (segment (start 70.761282 104.909291) (end 70.761282 107.191947) (width 0.6) (layer "B.Cu") (net 52))
   (segment (start 72.7 69.72) (end 72.7 68.971634) (width 1) (layer "B.Cu") (net 53))
   (segment (start 72.7 68.971634) (end 76.13157 65.540064) (width 1) (layer "B.Cu") (net 53))
